File: Lab 4/FINAL_DESIGN.sch (EAGLE design)
At the start: 49 parts, among them J1 FTDI_DEVICERA_SMT, M1 WIRELESS-NRF24L01, U1 3.3V, U2 GY-521MPU6050

Commit message: reconnected voltage regulator, added LEDs
Parts:
- removed R10, R11, R8: 10k, SparkFun-Resistors:2.2KOHM-0603-1/10W-1%
- added D1: Yellow, SparkFun-LED:LED-YELLOWLILYPAD
- C11, C12: value 100nF -> 100uF
- C13: value 100nF -> 0.1uF
- C14: value 100nF -> 4.7uF
- D2: device SparkFun-LED:LED-YELLOW0603 -> SparkFun-LED:LED-YELLOWLILYPAD
- L1: value 33nH/±5%/500mA -> 10uH
- R12, R9: value 10k -> 1k
Connections:
- net VR-LX renamed N$1
- removed net N$1 (its old number): C7.1, U1.AVCC
- removed net VR-FB: R8.1, R9.2, U$2.FB
- removed net VR-IN: C12.1, L1.1, R10.2, U$2.IN
- removed net VR-OUT: C14.1, R12.2, R8.2, U$2.OUT
- removed net VR-PGI: R10.1, R11.2, U$2.PGI
- removed net VR-~PGO: R12.1, U$2.~PGO
- new net IMU-INT: U1.PD3(INT1), U2.INT
- new net N$10: R12.2, U1.PC5(ADC5/SCL)
- new net N$8: D1.A, R9.1
- new net N$9: D2.A, R12.1
- net BATTERY+: now also C11.1, L1.1, U$2.IN
- net GND: now also U$2.FB, U$2.PGI, U$2.~PGO, U1.AGND; no longer R11.1, R9.1, U$2.3/~5
- net IMU-SCL: now also D2.C; no longer U1.PC5(ADC5/SCL)
- net IMU-SDA: now also D1.C; no longer U1.PC4(ADC4/SDA)
- net MEASURE_PIN: now also U1.PD4(XCK/T0); no longer U1.PD7(AIN1)
- net N$3: now also R9.2, U1.PC4(ADC4/SDA); no longer D2.C, S1.1
- net RESET: now also S1.1; no longer D2.A
- net VCC: now also C14.1, C7.1, U$2.OUT, U1.AVCC
- net VR-PS: now also C12.1, U$2.3/~5; no longer C13.1
- net VR-REF: now also C13.1; no longer C11.1
Other:
- moved on the sheet: C10, C11, C12, C13, C14, C6, C8, C9, D2, DIODE, DIODE1, DIODE2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

Commit message: Add new oscillator and wiring!!! Good work team!!
Parts:
- added C15: 100nF, SparkFun-Capacitors:0.1UF-25V(+80/-20%)(0603)
- U$3: value SIT8021SIT8021 -> LTC6930CMS8-8.19LTC6930CMS8-8.19; device SiT8021:SIT8021SIT8021 -> LTC6390:LTC6930CMS8-8.19LTC6930CMS8-8.19
Connections:
- net GND: now also C15.2, U$3.DIVA, U$3.DIVB, U$3.DIVC, U$3.GND2; no longer U$3.ST
- net VCC: now also C15.1, U$3.V+, U$3.V+2; no longer U$3.VDD
Changed lines of the file:
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@@
 <?xml version="1.0" encoding="utf-8"?>
 <!DOCTYPE eagle SYSTEM "eagle.dtd">
-<eagle version="8.4.1">
+<eagle version="8.4.3">
 <drawing>
 <settings>
@@
 <part name="DIODE4" library="quad" deviceset="DB2W40300L" device=""/>
 <part name="C11" library="SparkFun-Passives" deviceset="CAP" device="0603-CAP" value="100uF"/>
-<part name="U$3" library="SiT8021" deviceset="SIT8021" device="SIT8021"/>
 <part name="R9" library="SparkFun-Resistors" deviceset="2.2KOHM" device="-0603-1/10W-1%" value="1k"/>
 <part name="D1" library="SparkFun-LED" deviceset="LED-YELLOW" device="LILYPAD" value="Yellow"/>
 <part name="R12" library="SparkFun-Resistors" deviceset="2.2KOHM" device="-0603-1/10W-1%" value="1k"/>
 <part name="D2" library="SparkFun-LED" deviceset="LED-YELLOW" device="LILYPAD" value="Yellow"/>
+<part name="U$3" library="LTC6390" deviceset="LTC6930CMS8-8.19" device="LTC6930CMS8-8.19"/>
+<part name="C15" library="SparkFun-Capacitors" deviceset="0.1UF-25V(+80/-20%)(0603)" device="" value="100nF"/>
 </parts>
 <sheets>
@@
 <instance part="DIODE4" gate="G$1" x="-236.22" y="109.22" rot="MR270"/>
 <instance part="C11" gate="G$1" x="-317.5" y="104.14"/>
-<instance part="U$3" gate="G$1" x="-111.76" y="48.26"/>
 <instance part="R9" gate="G$1" x="-81.28" y="111.76" rot="R180"/>
 <instance part="D1" gate="G$1" x="-71.12" y="111.76" rot="R90"/>
 <instance part="R12" gate="G$1" x="-45.72" y="109.22" rot="R180"/>
 <instance part="D2" gate="G$1" x="-38.1" y="109.22" rot="R90"/>
+<instance part="U$3" gate="G$1" x="-99.06" y="38.1"/>
+<instance part="C15" gate="G$1" x="-55.88" y="38.1"/>
 </instances>
 <busses>
@@
 </segment>
 <segment>
-<pinref part="U$3" gate="G$1" pin="GND"/>
-<wire x1="-99.06" y1="53.34" x2="-83.82" y2="53.34" width="0.1524" layer="91"/>
-<label x="-88.9" y="53.34" size="1.778" layer="95"/>
-</segment>
-<segment>
-<pinref part="U$3" gate="G$1" pin="ST"/>
-<wire x1="-124.46" y1="53.34" x2="-134.62" y2="53.34" width="0.1524" layer="91"/>
-<label x="-134.62" y="53.34" size="1.778" layer="95"/>
-</segment>
-<segment>
 <pinref part="U$2" gate="G$1" pin="FB"/>
 <wire x1="-269.24" y1="53.34" x2="-254" y2="53.34" width="0.1524" layer="91"/>
@@
 <wire x1="-254" y1="30.48" x2="-254" y2="25.4" width="0.1524" layer="91"/>
 <label x="-254" y="25.4" size="1.778" layer="95"/>
+</segment>
+<segment>
+<pinref part="U$3" gate="G$1" pin="GND"/>
+<wire x1="-119.38" y1="43.18" x2="-129.54" y2="43.18" width="0.1524" layer="91"/>
+<label x="-129.54" y="43.18" size="1.778" layer="95"/>
+</segment>
+<segment>
+<pinref part="U$3" gate="G$1" pin="DIVA"/>
+<wire x1="-119.38" y1="33.02" x2="-129.54" y2="33.02" width="0.1524" layer="91"/>
+<label x="-129.54" y="33.02" size="1.778" layer="95"/>
+</segment>
+<segment>
+<pinref part="U$3" gate="G$1" pin="DIVB"/>
+<wire x1="-119.38" y1="27.94" x2="-129.54" y2="27.94" width="0.1524" layer="91"/>
+<label x="-129.54" y="27.94" size="1.778" layer="95"/>
+</segment>
+<segment>
+<pinref part="U$3" gate="G$1" pin="GND2"/>
+<wire x1="-78.74" y1="33.02" x2="-68.58" y2="33.02" width="0.1524" layer="91"/>
+<label x="-73.66" y="33.02" size="1.778" layer="95"/>
+</segment>
+<segment>
+<pinref part="U$3" gate="G$1" pin="DIVC"/>
+<wire x1="-78.74" y1="27.94" x2="-68.58" y2="27.94" width="0.1524" layer="91"/>
+<label x="-73.66" y="27.94" size="1.778" layer="95"/>
+</segment>
+<segment>
+<pinref part="C15" gate="G$1" pin="2"/>
+<wire x1="-55.88" y1="35.56" x2="-55.88" y2="25.4" width="0.1524" layer="91"/>
+<label x="-53.34" y="27.94" size="1.778" layer="95"/>
 </segment>
 </net>
@@
 </segment>
 <segment>
-<pinref part="U$3" gate="G$1" pin="VDD"/>
-<wire x1="-99.06" y1="43.18" x2="-83.82" y2="43.18" width="0.1524" layer="91"/>
-<label x="-88.9" y="43.18" size="1.778" layer="95"/>
-</segment>
-<segment>
 <pinref part="U$2" gate="G$1" pin="OUT"/>
 <wire x1="-269.24" y1="45.72" x2="-254" y2="45.72" width="0.1524" layer="91"/>
@@
 <pinref part="C14" gate="G$1" pin="1"/>
 <wire x1="-254" y1="45.72" x2="-254" y2="38.1" width="0.1524" layer="91"/>
+</segment>
+<segment>
+<pinref part="U$3" gate="G$1" pin="V+"/>
+<wire x1="-119.38" y1="48.26" x2="-129.54" y2="48.26" width="0.1524" layer="91"/>
+<label x="-129.54" y="48.26" size="1.778" layer="95"/>
+</segment>
+<segment>
+<pinref part="U$3" gate="G$1" pin="V+2"/>
+<wire x1="-78.74" y1="48.26" x2="-68.58" y2="48.26" width="0.1524" layer="91"/>
+<label x="-73.66" y="48.26" size="1.778" layer="95"/>
+</segment>
+<segment>
+<pinref part="C15" gate="G$1" pin="1"/>
+<wire x1="-55.88" y1="43.18" x2="-55.88" y2="50.8" width="0.1524" layer="91"/>
+<label x="-53.34" y="48.26" size="1.778" layer="95"/>
 </segment>
 </net>
@@
 <segment>
 <pinref part="U$3" gate="G$1" pin="OUT"/>
-<wire x1="-124.46" y1="43.18" x2="-134.62" y2="43.18" width="0.1524" layer="91"/>
-<label x="-134.62" y="43.18" size="1.778" layer="95"/>
-</segment>
-</net>
+<wire x1="-78.74" y1="43.18" x2="-68.58" y2="43.18" width="0.1524" layer="91"/>
+<label x="-76.2" y="43.18" size="1.778" layer="95"/>
+</segment>
+</net>

Commit message: CHANG FTDI connection according to Thomas: RX---RX TX-TX
Connections:
- net FTDI-RX: now also U1.PD0(RXD); no longer U1.PD1(TXD)
- net FTDI-TX: now also U1.PD1(TXD); no longer U1.PD0(RXD)
Changed lines of the file:
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@@
 </segment>
 <segment>
-<pinref part="U1" gate="U$1" pin="PD1(TXD)"/>
-<wire x1="-88.9" y1="96.52" x2="-83.82" y2="96.52" width="0.1524" layer="91"/>
-<label x="-86.36" y="96.52" size="1.778" layer="95"/>
+<pinref part="U1" gate="U$1" pin="PD0(RXD)"/>
+<wire x1="-88.9" y1="99.06" x2="-83.82" y2="99.06" width="0.1524" layer="91"/>
+<label x="-86.36" y="99.06" size="1.778" layer="95"/>
 </segment>
 </net>
@@
 </segment>
 <segment>
-<pinref part="U1" gate="U$1" pin="PD0(RXD)"/>
-<wire x1="-88.9" y1="99.06" x2="-83.82" y2="99.06" width="0.1524" layer="91"/>
-<label x="-86.36" y="99.06" size="1.778" layer="95"/>
+<pinref part="U1" gate="U$1" pin="PD1(TXD)"/>
+<wire x1="-88.9" y1="96.52" x2="-83.82" y2="96.52" width="0.1524" layer="91"/>
+<label x="-86.36" y="96.52" size="1.778" layer="95"/>
 </segment>
 </net>
