File: Lab 4/LATEST_DESIGN.sch (EAGLE design)
At the start: 46 parts, among them J1 FTDI_DEVICERA_SMT, M1 WIRELESS-NRF24L01, U1 3.3V, U2 GY-521MPU6050, U3 MAX7375AXR805-T

Commit message: MLF->TQFP, MOTOR1 now PWM, MP now analog
Parts:
- removed C4, C5, C7: 100nF, SparkFun-Passives:CAP0603-CAP
- removed D2: Yellow, SparkFun-LED:LED-YELLOWLILYPAD
- removed R12, R9: 1k, SparkFun-Resistors:2.2KOHM-0603-1/10W-1%
- removed U1: 3.3V, SparkFun-DigitalIC:ATMEGA328P_MLFMLF32
- added C13, C14, C16: 100nF, SparkFun-Passives:CAP0603-CAP
- added D3, D4: Yellow, SparkFun-LED:LED-YELLOWLILYPAD
- added R10, R8: 1k, SparkFun-Resistors:2.2KOHM-0603-1/10W-1%
- added R11: 10k, SparkFun-Resistors:2.2KOHM-0603-1/10W-1%
- added U4: ATMEGA328P_TQFP, quad:ATMEGA328P_TQFP
- R3: value 10k -> 1k
Connections:
- removed net BATTERY_+: C11.2
- removed net BATTER_+: L1.1, U$4.V_IN
- removed net N$10: R12.2, U1.PC5(ADC5/SCL)
- removed net N$8: D1.A, R9.1
- removed net N$9: D2.A, R12.1
- new net N$1: R8.2, U4.PC4(ADC4/SDA)
- new net N$11: D3.A, R8.1
- new net N$12: D4.A, R10.1
- new net N$14: R10.2, U4.PC5(ADC5/SCL)
- new net N$15: C13.1, U4.AREF
- net BATTERY+: now also C11.2, L1.1, U$4.V_IN
- net FTDI-RX: now also U4.PD0(RXD); no longer U1.PD0(RXD)
- net FTDI-TX: now also U4.PD1(TXD); no longer U1.PD1(TXD)
- net GND: now also C13.2, C14.2, C16.2, U3.GND, U4.AGND, U4.GND@3, U4.GND@5; no longer C4.2, C5.2, C7.2, U1.AGND, U1.GND@3, U1.GND@5, U1.GND@PAD
- net IMU-INT: now also D1.C; no longer U1.PD3(INT1)
- net IMU-SCL: now also D4.C; no longer D2.C
- net IMU-SDA: now also D3.C; no longer D1.C
- net MEASURE_PIN: now also U4.PC3(ADC3); no longer U1.PD4(XCK/T0)
- net MOTOR1: now also U4.PD3(INT1); no longer U1.PD2(INT0)
- net MOTOR2: now also U4.PD5(T1); no longer U1.PD5(T1)
- net MOTOR3: now also U4.PD6(AIN0); no longer U1.PD6(AIN0)
- net MOTOR4: now also U4.PB1(OC1A); no longer U1.PB1(OC1A)
- net N$2: now also R3.2, U4.PD2(INT0); no longer C4.1, U1.AREF
- net N$3: now also D1.A, R3.1; no longer R9.2, U1.PC4(ADC4/SDA)
- net OSC1: now also U4.PB6(XTAL1/TOSC1); no longer U1.PB6(XTAL1/TOSC1)
- net RESET: now also R11.1, U4.PC6(/RESET); no longer R3.1, U1.PC6(/RESET)
- net RF-CE: now also U4.PB0(ICP); no longer U1.PB0(ICP)
- net RF-CSN: now also U4.PB2(SS/OC1B); no longer U1.PB2(SS/OC1B)
- net RF-MISO: now also U4.PB4(MISO); no longer U1.PB4(MISO)
- net RF-MOSI: now also U4.PB3(MOSI/OC2); no longer U1.PB3(MOSI/OC2)
- net RF-SCK: now also U4.PB5(SCK); no longer U1.PB5(SCK)
- net VCC: now also C14.1, C16.1, R11.2, U4.AVCC, U4.VCC@4, U4.VCC@6; no longer C5.1, C7.1, R3.2, U1.AVCC, U1.VCC@4
Other:
- moved on the sheet: C10, C2, C3, D1, DIODE3, M1, NMOS3, R3, R7

Commit message: - Voltage Regulator: SEL, SHDN to GND - MCU: LEDs to GND - Replace 10muH Inductor schematic to match BOM (0603) - Replace 100uF Capacitors schematic to match BOM (1210)
Parts:
- removed C10, C12, C6, C8, C9: 100uF, SparkFun-Passives:CAP0603-CAP
- removed L1: 10uH, inductor-coilcraft:DO3316P
- added U$2, U$3, U$5, U$6, U$7: GRM31CD80J107ME39LGRM31CD80J107ME39L, GRM31CD80J107ME39L:GRM31CD80J107ME39LGRM31CD80J107ME39L
- added U$8: LQM18FN100M00DLQM18FN100M00D, LQM18FN100M00D:LQM18FN100M00DLQM18FN100M00D
Connections:
- net BATTERY+: now also U$2.P$1, U$3.P$1, U$5.P$1, U$6.P$1, U$8.P$1; no longer C10.2, C6.2, C8.2, C9.2, L1.1
- net GND: now also D1.C, D3.C, D4.C, U$2.P$2, U$3.P$2, U$4.SEL, U$4.SHDN, U$5.P$2, U$6.P$2, U$7.P$2; no longer C10.1, C12.1, C6.1, C8.1, C9.1
- net IMU-INT: no longer D1.C
- net IMU-SCL: no longer D4.C
- net IMU-SDA: no longer D3.C
- net VCC: now also U$7.P$1; no longer C12.2
- net VR_SW: now also U$8.P$2; no longer L1.2

Commit message: Packages: Ind, Cap. MCU: LEDs
100uF now 1206
10nH now 0603
LEDs pulled to ground
Parts:
- removed U$2, U$3, U$5, U$6, U$7: GRM31CD80J107ME39LGRM31CD80J107ME39L, GRM31CD80J107ME39L:GRM31CD80J107ME39LGRM31CD80J107ME39L
- removed U$8: LQM18FN100M00DLQM18FN100M00D, LQM18FN100M00D:LQM18FN100M00DLQM18FN100M00D
- added C10, C12, C6, C8, C9: 100uF, SparkFun-Passives:CAP1206
- added D2: BLUE, LEDs:LED-BLUE0603
- added L2: 10uH, SparkFun-Coils:INDUCTOR-0603-33NH
- added R9: 2.2k, SparkFun-Resistors:2.2KOHM-0603-1/10W-1%
- C11: device SparkFun-Passives:CAP0603-CAP -> SparkFun-Passives:CAP1206
- D1: value Yellow -> BLUE; device SparkFun-LED:LED-YELLOWLILYPAD -> LEDs:LED-BLUE0603; SPICEPREFIX (none) -> D
- D3, D4: value Yellow -> BLUE; device SparkFun-LED:LED-YELLOWLILYPAD -> LEDs:LED-BLUE0603
- R10, R8: value 1k -> 2.2k
- R3: value 1k -> 2.2k; SPICEPREFIX (none) -> R
Connections:
- removed net N$1 (its old number): R8.2, U4.PC4(ADC4/SDA)
- removed net N$11 (its old number): D3.A, R8.1
- removed net N$14: R10.2, U4.PC5(ADC5/SCL)
- removed net N$2: R3.2, U4.PD2(INT0)
- new net N$10: D2.A, R8.1
- new net N$3: D3.A, R9.1
- net BATTERY+: now also C10.2, C6.2, C8.2, C9.2, L2.1; no longer U$2.P$1, U$3.P$1, U$5.P$1, U$6.P$1, U$8.P$1
- net GND: now also C10.1, C12.1, C6.1, C8.1, C9.1, D2.C; no longer U$2.P$2, U$3.P$2, U$4.SEL, U$4.SHDN, U$5.P$2, U$6.P$2, U$7.P$2
- net IMU-INT: now also U4.PD2(INT0)
- net IMU-SCL: now also U4.PC5(ADC5/SCL)
- net IMU-SDA: now also U4.PC4(ADC4/SDA)
- net MOTOR1: now also R3.2
- net MOTOR2: now also R8.2
- net MOTOR3: now also R9.2
- net MOTOR4: now also R10.2
- net VCC: now also C12.2; no longer U$7.P$1
- net VR_SW: now also L2.2; no longer U$8.P$2
Other:
- moved on the sheet: R10, R3, R8

Commit message: Voltage regulator: SEL and SHDN to GND
Connections:
- net GND: now also U$4.SEL, U$4.SHDN
Changed lines of the file:
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@@
 <?xml version="1.0" encoding="utf-8"?>
 <!DOCTYPE eagle SYSTEM "eagle.dtd">
-<eagle version="8.4.1">
+<eagle version="8.4.3">
 <drawing>
 <settings>
@@
 <label x="-20.32" y="66.04" size="1.778" layer="95"/>
 </segment>
+<segment>
+<pinref part="U$4" gate="G$1" pin="SEL"/>
+<wire x1="-294.64" y1="86.36" x2="-302.26" y2="86.36" width="0.1524" layer="91"/>
+<label x="-304.8" y="86.36" size="1.778" layer="95"/>
+</segment>
+<segment>
+<pinref part="U$4" gate="G$1" pin="SHDN"/>
+<wire x1="-294.64" y1="76.2" x2="-302.26" y2="76.2" width="0.1524" layer="91"/>
+<label x="-304.8" y="76.2" size="1.778" layer="95"/>
+</segment>
 </net>
