File: Lab 5/PCBv1.brd (EAGLE design)
At the start: 100 x 80 mm, 48 parts, among them J1 FTDI_DEVICERA_SMT, M1 WIRELESS-NRF24L01, U1 3.3V, U2 GY-521MPU6050

Commit message: Update template
Parts:
- moved U$3 220.9 mm to (62.2, 69.8)
- moved NMOS2 159.7 mm to (62.2, 25.4)
- moved C6 153.8 mm to (49.5, 16.5)
- moved MOTOR 149.9 mm to (54.6, 36.8)
- moved NMOS1 149.5 mm to (62.2, 16.5)
- moved NMOS 134.0 mm to (63.5, 35.6)
- moved R6 127.3 mm to (58.4, 24.1)
- moved R5 126.9 mm to (58.4, 15.2)
- moved R7 125.9 mm to (58.4, 45.7)
- moved U$2 122.7 mm to (33.0, 25.4)
- moved U$1 121.3 mm to (90.2, 72.4)
- moved R4 117.0 mm to (58.4, 34.3)
- moved DIODE1 115.3 mm to (58.4, 19.1)
- moved DIODE2 114.9 mm to (58.4, 27.9)
- moved R9 114.5 mm to (44.4, 72.4)
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