File: Lab 5/template.brd (EAGLE design)
At the start: 100 x 80 mm, 48 parts, among them J1 FTDI_DEVICERA_SMT, M1 WIRELESS-NRF24L01, U1 3.3V, U2 GY-521MPU6050

Commit message: Update template
Parts:
- moved C15 87.3 mm to (67.3, 69.8)
- moved S1 27.1 mm to (8.86, 30.5)
- moved U$1 25.4 mm to (90.2, 72.4)
- moved U$3 16.5 mm to (62.2, 69.8)
- moved D2 1.27 mm to (38.1, 64.8)
- moved R12 1.27 mm to (33.0, 64.8)
- moved U1 1.27 mm to (36.8, 73.7)
- moved R3 1.27 mm to (43.2, 62.2)
- moved C4 1.27 mm to (40.6, 76.2)
- moved C5 1.27 mm to (33.0, 74.9)
- moved C7 1.27 mm to (40.6, 72.4)
- moved D1 1.27 mm to (43.2, 67.3)
- moved R9 1.27 mm to (44.4, 72.4)
