File: Lab 5/routev4.1.sch (EAGLE design)
At the start: 48 parts, among them J1 FTDI_DEVICE, M1 WIRELESS-NRF24L01, U2 GY-521MPU6050, U3 ATMEGA328P_TQFP

Commit message: routev4.1 idea crashed and burned: FTDI not the right module Ugggg; Update Template replacing with the correct one
Parts:
- renumbered J1 to J2
Changed lines of the file:
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@@
 <part name="C15" library="SparkFun-Capacitors" deviceset="0.1UF-25V(+80/-20%)(0603)" device="" value="100nF"/>
 <part name="U3" library="quad" deviceset="ATMEGA328P_TQFP" device="" value="ATMEGA328P_TQFP"/>
-<part name="J1" library="quad" deviceset="FTDI_DEVICE" device=""/>
+<part name="J2" library="quad" deviceset="FTDI_DEVICE" device=""/>
 </parts>
 <sheets>
@@
 <instance part="C15" gate="G$1" x="-55.88" y="38.1"/>
 <instance part="U3" gate="U$1" x="-111.76" y="91.44"/>
-<instance part="J1" gate="G$1" x="-193.04" y="121.92" rot="R180"/>
+<instance part="J2" gate="G$1" x="-193.04" y="121.92" rot="R180"/>
 </instances>
 <busses>
@@
 <wire x1="-187.96" y1="129.54" x2="-182.88" y2="129.54" width="0.1524" layer="91"/>
 <label x="-187.96" y="129.54" size="1.778" layer="95"/>
-<pinref part="J1" gate="G$1" pin="GND"/>
+<pinref part="J2" gate="G$1" pin="GND"/>
 </segment>
 <segment>
@@
 <wire x1="-187.96" y1="121.92" x2="-182.88" y2="121.92" width="0.1524" layer="91"/>
 <label x="-187.96" y="121.92" size="1.778" layer="95"/>
-<pinref part="J1" gate="G$1" pin="RXI"/>
+<pinref part="J2" gate="G$1" pin="RXI"/>
 </segment>
 <segment>
@@
 <wire x1="-187.96" y1="119.38" x2="-182.88" y2="119.38" width="0.1524" layer="91"/>
 <label x="-187.96" y="119.38" size="1.778" layer="95"/>
-<pinref part="J1" gate="G$1" pin="TXO"/>
+<pinref part="J2" gate="G$1" pin="TXO"/>
 </segment>
 <segment>
@@
 <wire x1="-187.96" y1="124.46" x2="-182.88" y2="124.46" width="0.1524" layer="91"/>
 <label x="-187.96" y="124.46" size="1.778" layer="95"/>
-<pinref part="J1" gate="G$1" pin="VCC"/>
+<pinref part="J2" gate="G$1" pin="VCC"/>
 </segment>
 <segment>
@@
 <segment>
 <pinref part="C1" gate="G$1" pin="1"/>
-<pinref part="J1" gate="G$1" pin="DTR"/>
-</segment>
-</net>
+<pinref part="J2" gate="G$1" pin="DTR"/>
+</segment>
+</net>
