File: Lab 5/routev10.1.brd (EAGLE design)
At the start: 100 x 80 mm, 48 parts, among them J1 FTDI_DEVICE, M1 WIRELESS-NRF24L01, U2 GY-521MPU6050, U3 ATMEGA328P_TQFP

Commit message: We need a redesign guys
Parts:
- removed J1: FTDI_DEVICE, quad:FTDI_DEVICE_SIDE
- removed U$3: LTC6930CMS8-8.19LTC6930CMS8-8.19, LTC6390:SOP65P490X110-8N
- added AXR1: MAX7375, quad:SC70-3L
- added J2: FTDI_DEVICE, quad:FTDI_DEVICE_SIDE
- C1: device SparkFun-Passives:0603-CAP -> SparkFun-Capacitors:0603-CAP
- R3: value 1k -> 10k
- moved L1 32.0 mm to (14.5, 36.1)
- moved U$1 28.7 mm to (2.87, 17.1), turned to 0 degrees
- moved C11 26.5 mm to (20.0, 30.6)
- moved C3 25.3 mm to (41.1, 9.70), turned to 90 degrees
- moved R1 25.3 mm to (25.4, 31.0), turned to 0 degrees
- moved C2 24.9 mm to (41.1, 6.65), turned to 90 degrees
- moved U$2 24.0 mm to (20.1, 34.0), turned to 0 degrees
- moved DIODE4 23.8 mm to (13.7, 33.4), turned to 180 degrees
- moved R2 23.5 mm to (29.2, 31.0)
- moved C14 22.9 mm to (25.8, 35.6), turned to 90 degrees
- moved C15 22.8 mm to (28.9, 28.7), turned to 90 degrees
- moved C12 21.2 mm to (15.6, 33.4), turned to 90 degrees
- moved R3 16.4 mm to (30.6, 8.18), turned to 0 degrees
- moved C4 15.6 mm to (16.4, 4.34), turned to 270 degrees
- moved U3 15.0 mm to (22.7, 6.36), turned to 270 degrees
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Connections:
- removed net N$13: C1.1, J1.P$1
- new net N$12: C1.1, J2.P$1
- net FTDI-RX: now also J2.P$3; no longer J1.P$3
- net FTDI-TX: now also J2.P$2; no longer J1.P$2
- net GND: now also AXR1.3, J2.P$6; no longer J1.P$6, U$3.2, U$3.3, U$3.4, U$3.5, U$3.6
- net N$1: now also U$2.16
- net OSC1: now also AXR1.2; no longer U$3.7
- net RESET: now also R3.1; no longer R3.2
- net VCC: now also AXR1.1, J2.P$4, R3.2, U3.6; no longer J1.P$4, R3.1, U$3.1, U$3.8
Routing:
- net N$11: track 163.0 -> 0.00 mm
- net BATTERY+: track 99.2 -> 0.00 mm, vias 2 -> 0
- net VCC: track 113.2 -> 156.9 mm, vias 4 -> 0
- net N$10: track 47.2 -> 16.4 mm
- net IMU-INT: track 45.0 -> 15.4 mm
- net N$8: track 41.6 -> 20.7 mm
- net RF-MOSI: track 12.3 -> 25.2 mm, vias 0 -> 1
- net RESET: track 21.3 -> 8.53 mm
- net RF-MISO: track 16.7 -> 29.0 mm, vias 2 -> 1
- net VR-PS: track 17.4 -> 6.08 mm, vias 0 -> 2
- net MEASURE_PIN: track 23.1 -> 34.1 mm
- net N$4: track 10.7 -> 0.00 mm
- net MOTOR4: track 10.5 -> 0.00 mm, vias 2 -> 0
- net N$12: track 0.00 -> 9.25 mm, vias 0 -> 1
- net IMU-SDA: track 14.9 -> 24.1 mm, vias 0 -> 2
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- removed copper zone on layer 1, net BATTERY_+
- removed copper zone on layer 16, net GND
- removed copper zone on layer 1, net S$1
- removed copper zone on layer 1, net S$2
Other:
- outline, holes or cut-outs redrawn
