File: Lab 5/routev7.5.brd (EAGLE design)
At the start: 100 x 80 mm, 48 parts, among them J1 FTDI_DEVICE, M1 WIRELESS-NRF24L01, U2 GY-521MPU6050, U3 ATMEGA328P_TQFP

Commit message: We need a redesign guys
Routing:
- added copper zone on layer 1, net BATTERY+
- added copper zone on layer 1, net VCC
- removed copper zone on layer 1, net BATTERY_+
- removed copper zone on layer 1, net S$1
- removed copper zone on layer 1, net S$2
Changed lines of the file:
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@@
 <wire x1="29.6926" y1="26.67" x2="30.187" y2="26.1756" width="0.8128" layer="1"/>
 <wire x1="30.187" y1="26.1756" x2="30.187" y2="24.5618" width="0.8128" layer="1"/>
+<polygon width="0.3048" layer="1">
+<vertex x="5.3594" y="28.0924"/>
+<vertex x="36.5506" y="28.0924"/>
+<vertex x="36.4744" y="9.0424"/>
+<vertex x="18.8468" y="9.0424"/>
+<vertex x="18.923" y="6.6294"/>
+<vertex x="18.6944" y="6.6294"/>
+<vertex x="18.6944" y="0"/>
+<vertex x="5.3594" y="0"/>
+</polygon>
 </signal>
 <signal name="RF-CE">
@@
 <wire x1="4.318" y1="19.8628" x2="3.23580625" y2="19.8628" width="0.8128" layer="1"/>
 <wire x1="3.23580625" y1="19.8628" x2="1.59385" y2="21.50475625" width="0.8128" layer="1"/>
+<polygon width="0.3048" layer="1">
+<vertex x="0" y="28.0416"/>
+<vertex x="4.8514" y="28.0162"/>
+<vertex x="4.8514" y="2.5654"/>
+<vertex x="0" y="2.5908"/>
+</polygon>
+<polygon width="0.3048" layer="1">
+<vertex x="19.4564" y="8.5344"/>
+<vertex x="31.1404" y="8.5344"/>
+<vertex x="31.1404" y="0.0508"/>
+<vertex x="19.4564" y="0.0508"/>
+</polygon>
 </signal>
 <signal name="N$5">
@@
 <wire x1="16.9164" y1="21.6408" x2="15.5956" y2="21.6408" width="0.3048" layer="16"/>
 </signal>
-<signal name="S$1">
-<polygon width="0.3048" layer="1">
-<vertex x="19.4564" y="8.5344"/>
-<vertex x="31.1404" y="8.5344"/>
-<vertex x="31.1404" y="0.0508"/>
-<vertex x="19.4564" y="0.0508"/>
-</polygon>
-</signal>
-<signal name="BATTERY_+">
-<polygon width="0.3048" layer="1">
-<vertex x="0" y="28.0416"/>
-<vertex x="4.8514" y="28.0162"/>
-<vertex x="4.8514" y="2.5654"/>
-<vertex x="0" y="2.5908"/>
-</polygon>
-</signal>
-<signal name="S$2">
-<polygon width="0.3048" layer="1">
-<vertex x="5.3594" y="28.0924"/>
-<vertex x="36.5506" y="28.0924"/>
-<vertex x="36.4744" y="9.0424"/>
-<vertex x="18.8468" y="9.0424"/>
-<vertex x="18.923" y="6.6294"/>
-<vertex x="18.6944" y="6.6294"/>
-<vertex x="18.6944" y="0"/>
-<vertex x="5.3594" y="0"/>
-</polygon>
-</signal>
 <signal name="N$13">
