File: Lab 5/routev8.2.brd (EAGLE design)
At the start: 100 x 80 mm, 48 parts, among them J1 FTDI_DEVICE, M1 WIRELESS-NRF24L01, U2 GY-521MPU6050, U3 ATMEGA328P_TQFP

Commit message: We need a redesign guys
Parts:
- removed J1: FTDI_DEVICE, quad:FTDI_DEVICE_SIDE
- added J2: FTDI_DEVICE, quad:FTDI_DEVICE_SIDE
- C1: device SparkFun-Passives:0603-CAP -> SparkFun-Capacitors:0603-CAP
- R3: value 1k -> 10k
- moved U$1 28.7 mm to (2.87, 17.1), turned to 0 degrees
- moved L1 26.3 mm to (6.55, 20.8)
- moved C3 25.3 mm to (41.1, 9.70), turned to 270 degrees
- moved C2 24.9 mm to (41.1, 6.65)
- moved DIODE4 23.2 mm to (5.54, 18.1), turned to 180 degrees
- moved C12 21.2 mm to (7.44, 18.1), turned to 90 degrees
- moved C11 19.9 mm to (11.9, 15.4)
- moved C5 18.4 mm to (32.9, 2.51), turned to 270 degrees
- moved U$2 17.2 mm to (12.0, 18.8), turned to 0 degrees
- moved R3 16.4 mm to (30.7, 8.18), turned to 0 degrees
- moved C7 16.1 mm to (32.7, 4.70), turned to 180 degrees
- moved C4 15.6 mm to (16.4, 4.34)
- moved U3 15.0 mm to (22.7, 6.36), turned to 270 degrees
- moved M1 14.2 mm to (25.5, 8.39), turned to 180 degrees
- moved MOTOR3 13.9 mm to (7.70, 2.92)
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Connections:
- removed net N$13: C1.1, J1.P$1
- new net N$12: C1.1, J2.P$1
- net FTDI-RX: now also J2.P$3; no longer J1.P$3
- net FTDI-TX: now also J2.P$2; no longer J1.P$2
- net GND: now also J2.P$6; no longer J1.P$6
- net RESET: now also R3.1; no longer R3.2
- net VCC: now also J2.P$4, R3.2; no longer J1.P$4, R3.1
Routing:
- net N$11: track 163.0 -> 0.00 mm
- net VCC: track 113.2 -> 0.00 mm, vias 4 -> 0
- net GND: track 111.0 -> 0.00 mm, vias 15 -> 0
- net BATTERY+: track 99.2 -> 25.3 mm, vias 2 -> 0
- net N$12: track 0.00 -> 47.4 mm, vias 0 -> 1
- net N$10: track 47.2 -> 16.4 mm
- net IMU-INT: track 45.0 -> 15.4 mm
- net MOTOR1: track 6.38 -> 30.4 mm, vias 0 -> 2
- net N$8: track 41.6 -> 20.7 mm
- net RESET: track 21.3 -> 39.7 mm, vias 0 -> 2
- net RF-MOSI: track 12.3 -> 25.2 mm, vias 0 -> 1
- net RF-MISO: track 16.7 -> 29.0 mm, vias 2 -> 1
- net IMU-SDA: track 14.9 -> 24.1 mm, vias 0 -> 1
- net MOTOR2: track 5.30 -> 14.5 mm
- net N$13: track 8.69 -> 0.00 mm, vias 2 -> 0
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- added copper zone on layer 1, net BATTERY+
- removed copper zone on layer 1, net BATTERY_+
- removed copper zone on layer 16, net GND
- removed copper zone on layer 1, net S$1
- removed copper zone on layer 1, net S$2
Other:
- outline, holes or cut-outs redrawn
