File: Lab 5/template.sch (EAGLE design)
At the start: 48 parts, among them J1 FTDI_DEVICE, M1 WIRELESS-NRF24L01, U2 GY-521MPU6050, U3 ATMEGA328P_TQFP

Commit message: Update template.sch
Parts:
- removed C11, C12: 100uF, SparkFun-Passives:CAP0603-CAP
- removed DIODE4: DB2W40300L, quad:DB2W40300L
- removed L1: 10uH, SparkFun-Coils:INDUCTOR-0603-33NH
- removed MOTOR: JST_CONNECTOR_FEMALE, quad:JST_CONNECTOR_FEMALE
- removed R12: 1k, SparkFun-Resistors:2.2KOHM-0603-1/10W-1%
- removed U$2: MAX1672'MAX1672', voltreg:MAX1672'MAX1672'
- removed U$3: LTC6930CMS8-8.19LTC6930CMS8-8.19, LTC6390:LTC6930CMS8-8.19LTC6930CMS8-8.19
- added C16: 100nF, SparkFun-Passives:CAP0603-CAP
- added D3, D4: BLUE, LEDs:LED-BLUE0603
- added IC1: MCP1253-ADJ, microchip:MCP1253-ADJ
- added MOTOR4: JST_CONNECTOR_FEMALE, quad:JST_CONNECTOR_FEMALE
- added R10, R8: 2.2k, SparkFun-Resistors:2.2KOHM-0603-1/10W-1%
- added R11: 10k, SparkFun-Resistors:2.2KOHM-0603-1/10W-1%
- added U4: ATMEGA328P_TQFP, quad:ATMEGA328P_TQFP
- C10, C6, C8, C9: device SparkFun-Passives:CAP0603-CAP -> SparkFun-Passives:CAP1206
- C13: value 0.1uF -> 100nF
- C14: value 4.7uF -> 100nF
- C4: value 100nF -> 1uF; device SparkFun-Passives:CAP0603-CAP -> SparkFun-Capacitors:0.1UF-25V(+80/-20%)(0603)
- C5, C7: value 100nF -> 10uF; device SparkFun-Passives:CAP0603-CAP -> SparkFun-Capacitors:0.1UF-25V(+80/-20%)(0603)
- D1: value Yellow -> BLUE; device SparkFun-LED:LED-YELLOWLILYPAD -> LEDs:LED-BLUE0603; SPICEPREFIX (none) -> D
- D2: value Yellow -> BLUE; device SparkFun-LED:LED-YELLOWLILYPAD -> LEDs:LED-BLUE0603
- R3: value 10k -> 2.2k; SPICEPREFIX (none) -> R
- R9: value 1k -> 2.2k
- U3: value ATMEGA328P_TQFP -> MAX7375AXR805-T; device quad:ATMEGA328P_TQFP -> MAX7375AXR805-T:MAX7375AXR805-T
Connections:
- removed net N$2 (its old number): C4.1, U3.AREF
- removed net VR-PS: C12.1, DIODE4.GPIN, U$2.3/~5, U$2.PS
- removed net VR-REF: C13.1, U$2.REF
- new net N$11: D1.A, R3.1
- new net N$15: C13.1, U4.AREF
- net BATTERY+: now also C7.2, IC1.FB, IC1.SHDN, IC1.VIN, MOTOR4.+; no longer C11.1, L1.1, MOTOR.+, U$2.IN
- net FTDI-RX: now also U4.PD0(RXD); no longer U3.PD0(RXD)
- net FTDI-TX: now also U4.PD1(TXD); no longer U3.PD1(TXD)
- net GND: now also C16.2, C7.1, D1.C, D2.C, D3.C, D4.C, IC1.GND, U3.GND, U4.AGND, U4.GND@3, U4.GND@5; no longer C11.2, C12.2, C4.2, C5.2, C7.2, U$2.FB, U$2.GND, U$2.PGI, U$2.PGND, U$2.~PGO, U$3.DIVA, U$3.DIVB, U$3.DIVC, U$3.GND, U$3.GND2, U3.AGND, U3.GND@3, U3.GND@5
- net IMU-INT: now also U4.PD2(INT0); no longer U3.PD3(INT1)
- net IMU-SCL: now also U4.PC5(ADC5/SCL); no longer D2.C
- net IMU-SDA: now also U4.PC4(ADC4/SDA); no longer D1.C
- net MEASURE_PIN: now also U4.PC3(ADC3); no longer U3.PD4(XCK/T0)
- net MOTOR1: now also R3.2, U4.PD3(INT1); no longer U3.PD2(INT0)
- net MOTOR2: now also R8.2, U4.PD5(T1); no longer U3.PD5(T1)
- net MOTOR3: now also R9.2, U4.PD6(AIN0); no longer U3.PD6(AIN0)
- net MOTOR4: now also R10.2, U4.PB1(OC1A); no longer U3.PB1(OC1A)
- net N$1: now also D4.A, R10.1; no longer DIODE4.PPIN, L1.2, U$2.LX
- net N$10: now also D2.A, R8.1; no longer R12.2, U3.PC5(ADC5/SCL)
- net N$3: now also D3.A; no longer D1.A
- net N$4: now also MOTOR2.-; no longer MOTOR1.-
- net N$5: now also MOTOR3.-; no longer MOTOR2.-
- net N$6: now also MOTOR1.-; no longer MOTOR.-
- net N$7: now also MOTOR4.-; no longer MOTOR3.-
- net N$8: now also C4.1, IC1.C-; no longer R9.2, U3.PC4(ADC4/SDA)
- net N$9: now also C4.2, IC1.C+; no longer D2.A, R12.1
- net OSC1: now also U3.CLOCK, U4.PB6(XTAL1/TOSC1); no longer U$3.OUT, U3.PB6(XTAL1/TOSC1)
- net RESET: now also R11.1, U4.PC6(/RESET); no longer R3.1, U3.PC6(/RESET)
- net RF-CE: now also U4.PB0(ICP); no longer U3.PB0(ICP)
- net RF-CSN: now also U4.PB2(SS/OC1B); no longer U3.PB2(SS/OC1B)
- net RF-MISO: now also U4.PB4(MISO); no longer U3.PB4(MISO)
- net RF-MOSI: now also U4.PB3(MOSI/OC2); no longer U3.PB3(MOSI/OC2)
- net RF-SCK: now also U4.PB5(SCK); no longer U3.PB5(SCK)
- net VCC: now also C16.1, IC1.VOUT, R11.2, U3.V+, U4.AVCC, U4.VCC@4, U4.VCC@6; no longer C5.1, C7.1, R3.2, U$2.OUT, U$3.V+, U$3.V+2, U3.AVCC, U3.VCC@4
Other:
- moved on the sheet: C10, C13, C14, C15, C2, C3, C4, C5, C7, DIODE3, M1, NMOS3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
