File: Lab 5/failed design/template.brd (EAGLE design)
At the start: 100 x 80 mm, 49 parts, among them IC1 MCP1253-ADJ, J1 FTDI_DEVICE, M1 WIRELESS-NRF24L01, U2 GY-521MPU6050, U3 MAX7375AXR805-T, U4 ATMEGA328P_TQFP

Commit message: Update template.sch
Parts:
- removed C16: 100nF, SparkFun-Passives:0603-CAP
- removed D3, D4: BLUE, LEDs:LED-0603
- removed IC1: MCP1253-ADJ, microchip:MSOP8
- removed R10, R8: 2.2k, SparkFun-Resistors:0603
- removed R11: 10k, SparkFun-Resistors:0603
- removed U4: ATMEGA328P_TQFP, quad:TQFP32-08
- added C11, C12: 100uF, SparkFun-Passives:0603-CAP
- added DIODE4: DB2W40300L, quad:MINI2-F3-B
- added L1: 10uH, SparkFun-Coils:0603
- added R12: 1k, SparkFun-Resistors:0603
- added U$2: MAX1672'MAX1672', voltreg:21-0055H_16
- added U$3: LTC6930CMS8-8.19LTC6930CMS8-8.19, LTC6390:SOP65P490X110-8N
- C10, C6, C8, C9: device SparkFun-Passives:1206 -> SparkFun-Passives:0603-CAP
- C13: value 100nF -> 0.1uF
- C14: value 100nF -> 4.7uF
- C4: value 1uF -> 100nF; device SparkFun-Capacitors:0603-CAP -> SparkFun-Passives:0603-CAP
- C5, C7: value 10uF -> 100nF; device SparkFun-Capacitors:0603-CAP -> SparkFun-Passives:0603-CAP
- D1, D2: value BLUE -> Yellow; device LEDs:LED-0603 -> SparkFun-LED:LED-1206
- R3: value 2.2k -> 10k
- R9: value 2.2k -> 1k
- U3: value MAX7375AXR805-T -> ATMEGA328P_TQFP; device MAX7375AXR805-T:21-0075D -> quad:TQFP32-08
- moved U$1 155.8 mm to (90.2, 72.4)
- moved C14 143.0 mm to (93.3, 10.5)
- moved C7 141.8 mm to (40.6, 72.4), turned to 90 degrees
- moved C4 139.5 mm to (40.6, 76.2), turned to 90 degrees
- moved C5 135.1 mm to (33.0, 74.9), turned to 90 degrees
- moved C13 133.8 mm to (88.2, 13.1)
- moved J1 130.2 mm to (87.5, 51.5)
- moved S1 120.0 mm to (90.1, 59.7)
- moved DIODE2 117.3 mm to (58.4, 27.9)
- moved NMOS2 116.9 mm to (62.2, 25.4)
- moved DIODE1 115.9 mm to (58.4, 19.1)
- moved C15 113.7 mm to (67.3, 69.8), turned to 270 degrees
- moved C1 111.8 mm to (85.1, 58.4)
- moved DIODE 111.7 mm to (58.4, 38.1)
- moved MOTOR4 110.3 mm to (54.6, 48.3)
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Connections:
- removed net N$11: D1.A, R3.1
- removed net N$15: C13.1, U4.20
- new net N$2: C4.1, U3.20
- new net VR-PS: C12.1, DIODE4.NEG, U$2.11, U$2.5
- new net VR-REF: C13.1, U$2.13
- net BATTERY+: now also C11.1, L1.1, U$2.12; no longer C7.2, IC1.3, IC1.7, IC1.8
- net FTDI-RX: now also U3.30; no longer U4.30
- net FTDI-TX: now also U3.31; no longer U4.31
- net GND: now also C11.2, C12.2, C4.2, C5.2, C7.2, U$2.10, U$2.14, U$2.2, U$2.6, U$2.7, U$3.2, U$3.3, U$3.4, U$3.5, U$3.6, U3.21, U3.5; no longer C16.2, C7.1, D1.C, D2.C, D3.C, D4.C, IC1.4, U4.21, U4.3, U4.5
- net IMU-INT: now also U3.1; no longer U4.32
- net IMU-SCL: now also D2.C; no longer U4.28
- net IMU-SDA: now also D1.C; no longer U4.27
- net MEASURE_PIN: now also U3.2; no longer U4.26
- net MOTOR1: now also U3.32; no longer R3.2, U4.1
- net MOTOR2: now also U3.9; no longer R8.2, U4.9
- net MOTOR3: now also U3.10; no longer R9.2, U4.10
- net MOTOR4: now also U3.13; no longer R10.2, U4.13
- net N$1: now also DIODE4.POS, L1.2, U$2.1, U$2.16; no longer D4.A, R10.1
- net N$10: now also R12.2, U3.28; no longer D2.A, R8.1
- net N$3: now also D1.A; no longer D3.A
- net N$8: now also R9.2, U3.27; no longer C4.1, IC1.5
- net N$9: now also D2.A, R12.1; no longer C4.2, IC1.6
- net OSC1: now also U$3.7, U3.7; no longer U3.2, U4.7
- net RESET: now also R3.1, U3.29; no longer R11.1, U4.29
- net RF-CE: now also U3.12; no longer U4.12
- net RF-CSN: now also U3.14; no longer U4.14
- net RF-MISO: now also U3.16; no longer U4.16
- net RF-MOSI: now also U3.15; no longer U4.15
- net RF-SCK: now also U3.17; no longer U4.17
- net VCC: now also C5.1, C7.1, R3.2, U$2.9, U$3.1, U$3.8, U3.18, U3.4; no longer C16.1, IC1.2, R11.2, U3.1, U4.18, U4.4, U4.6
Routing:
- net N$11: track 0.00 -> 166.0 mm
