File: Lab 5/failed design/template.sch (EAGLE design)
At the start: 45 parts, among them J1 FTDI_DEVICE, M1 WIRELESS-NRF24L01, U2 GY-521MPU6050, U3 MAX7375AXR805-T, U4 ATMEGA328P_TQFP

Commit message: Update template.sch
Parts:
- removed C16: 100nF, SparkFun-Passives:CAP0603-CAP
- removed D3, D4: BLUE, LEDs:LED-BLUE0603
- removed R10, R8: 2.2k, SparkFun-Resistors:2.2KOHM-0603-1/10W-1%
- removed R11: 10k, SparkFun-Resistors:2.2KOHM-0603-1/10W-1%
- removed U4: ATMEGA328P_TQFP, quad:ATMEGA328P_TQFP
- added C11, C12: 100uF, SparkFun-Passives:CAP0603-CAP
- added C4, C5, C7: 100nF, SparkFun-Passives:CAP0603-CAP
- added DIODE4: DB2W40300L, quad:DB2W40300L
- added L1: 10uH, SparkFun-Coils:INDUCTOR-0603-33NH
- added R12: 1k, SparkFun-Resistors:2.2KOHM-0603-1/10W-1%
- added U$2: MAX1672'MAX1672', voltreg:MAX1672'MAX1672'
- added U$3: LTC6930CMS8-8.19LTC6930CMS8-8.19, LTC6390:LTC6930CMS8-8.19LTC6930CMS8-8.19
- C10, C6, C8, C9: device SparkFun-Passives:CAP1206 -> SparkFun-Passives:CAP0603-CAP
- C13: value 100nF -> 0.1uF
- C14: value 100nF -> 4.7uF
- D1: value BLUE -> Yellow; device LEDs:LED-BLUE0603 -> SparkFun-LED:LED-YELLOWLILYPAD; SPICEPREFIX D -> (none)
- D2: value BLUE -> Yellow; device LEDs:LED-BLUE0603 -> SparkFun-LED:LED-YELLOWLILYPAD
- R3: value 2.2k -> 10k; SPICEPREFIX R -> (none)
- R9: value 2.2k -> 1k
- U3: value MAX7375AXR805-T -> ATMEGA328P_TQFP; device MAX7375AXR805-T:MAX7375AXR805-T -> quad:ATMEGA328P_TQFP
Connections:
- removed net N$11: D1.A, R3.1
- removed net N$15: C13.1, U4.AREF
- new net N$2: C4.1, U3.AREF
- new net N$8: R9.2, U3.PC4(ADC4/SDA)
- new net N$9: D2.A, R12.1
- new net VR-PS: C12.1, DIODE4.GPIN, U$2.3/~5, U$2.PS
- new net VR-REF: C13.1, U$2.REF
- net BATTERY+: now also C11.1, L1.1, U$2.IN
- net FTDI-RX: now also U3.PD0(RXD); no longer U4.PD0(RXD)
- net FTDI-TX: now also U3.PD1(TXD); no longer U4.PD1(TXD)
- net GND: now also C11.2, C12.2, C4.2, C5.2, C7.2, U$2.FB, U$2.GND, U$2.PGI, U$2.PGND, U$2.~PGO, U$3.DIVA, U$3.DIVB, U$3.DIVC, U$3.GND, U$3.GND2, U3.AGND, U3.GND@3, U3.GND@5; no longer C16.2, D1.C, D2.C, D3.C, D4.C, U3.GND, U4.AGND, U4.GND@3, U4.GND@5
- net IMU-INT: now also U3.PD3(INT1); no longer U4.PD2(INT0)
- net IMU-SCL: now also D2.C; no longer U4.PC5(ADC5/SCL)
- net IMU-SDA: now also D1.C; no longer U4.PC4(ADC4/SDA)
- net MEASURE_PIN: now also U3.PD4(XCK/T0); no longer U4.PC3(ADC3)
- net MOTOR1: now also U3.PD2(INT0); no longer R3.2, U4.PD3(INT1)
- net MOTOR2: now also U3.PD5(T1); no longer R8.2, U4.PD5(T1)
- net MOTOR3: now also U3.PD6(AIN0); no longer R9.2, U4.PD6(AIN0)
- net MOTOR4: now also U3.PB1(OC1A); no longer R10.2, U4.PB1(OC1A)
- net N$1: now also DIODE4.PPIN, L1.2, U$2.LX, U$2.LX1; no longer D4.A, R10.1
- net N$10: now also R12.2, U3.PC5(ADC5/SCL); no longer D2.A, R8.1
- net N$3: now also D1.A; no longer D3.A
- net OSC1: now also U$3.OUT, U3.PB6(XTAL1/TOSC1); no longer U3.CLOCK, U4.PB6(XTAL1/TOSC1)
- net RESET: now also R3.1, U3.PC6(/RESET); no longer R11.1, U4.PC6(/RESET)
- net RF-CE: now also U3.PB0(ICP); no longer U4.PB0(ICP)
- net RF-CSN: now also U3.PB2(SS/OC1B); no longer U4.PB2(SS/OC1B)
- net RF-MISO: now also U3.PB4(MISO); no longer U4.PB4(MISO)
- net RF-MOSI: now also U3.PB3(MOSI/OC2); no longer U4.PB3(MOSI/OC2)
- net RF-SCK: now also U3.PB5(SCK); no longer U4.PB5(SCK)
- net VCC: now also C5.1, C7.1, R3.2, U$2.OUT, U$3.V+, U$3.V+2, U3.AVCC, U3.VCC@4; no longer C16.1, R11.2, U3.V+, U4.AVCC, U4.VCC@4, U4.VCC@6
Other:
- moved on the sheet: C10, C13, C14, C15, C2, C3, DIODE3, M1, NMOS3, R3, R7, R9
